Commit message: Gazebo: realistic fruited plants, clear the aisles, ghost robot (no tipping)
Fixes the robot tipping/wedging seen in Gazebo and the patrol timeouts.

- Root cause of the freeze: the 0.30 m red crates sat inside the 0.8 m
  driving aisles. The robot drove onto one, climbed and tipped; once
  pitched, VelocityControl froze it there and no goal could be reached.
- Remove the crates entirely -- the fruited plants are now the harvest
  targets, nothing blocks the aisles.
- Richer strawberry plants: brown pot + bushy green foliage + 6 ripe red
  berries each, 9 plants per gutter (kept well above the 0.20 m lidar
  plane so they never clutter the map).
- Robot is now a kinematic 'ghost': removed the base collision and
  disabled gravity, so VelocityControl glides it level in the plane and
  it can never tip or wedge on the geometry (matches the headless model).

Co-Authored-By: Claude Opus 4.8 <noreply@anthropic.com>
Claude-Session: https://claude.ai/code/session_01Uhu7fuqyazcPGV5GTXJMX5

File: src/youbot_gazebo/urdf/youbot_gz.urdf (robot description, URDF)
Before this commit: robot youbot, 8 links, 7 joints
Links:
- link base_link: geometry visual box size=0.28 0.34 0.03; visual box size=0.57 0.36 0.10

Commit message: Add RGB camera + colour-based strawberry detection in Gazebo
- youbot_gz.urdf: front camera on a short mast (0.55 m, tipped 0.15 rad
  down), gz camera sensor -> /camera image + camera_info.
- gz_bridge.yaml: bridge /camera/image and /camera/camera_info to ROS.
- strawberry_detector node (youbot_control): segments ripe (near-pure-red)
  fruit with lib/vision.red_mask, draws green boxes on the frame, publishes
  /camera/detections (annotated Image) and /ripe_count. Same node interface
  a YOLOv8 model would later drop into for real-world robustness.
- gazebo.launch.py: run the detector alongside the control stack.
- mission_node: bump goal timeout 45 -> 60 s for the long depot diagonal.

Colour detection is the pragmatic choice for the digital twin (berries are
near-pure red); ML (YOLOv8) is the deployment path, swappable without
touching the rest of the stack.

Co-Authored-By: Claude Opus 4.8 <noreply@anthropic.com>
Claude-Session: https://claude.ai/code/session_01Uhu7fuqyazcPGV5GTXJMX5

File: src/youbot_gazebo/urdf/youbot_gz.urdf (robot description, URDF)
Before this commit: robot youbot, 8 links, 7 joints
Links:
- added link camera, mass 0.05; visual box size=0.03 0.09 0.03
- added link mast, mass 0.1; visual cylinder length=0.38 radius=0.015
Joints:
- added joint j_camera: type fixed, parent base_link, child camera, origin xyz=0.24 0 0.55 rpy=0 0.15 0
- added joint j_mast: type fixed, parent base_link, child mast, origin xyz=0.22 0 0.16

Commit message: Camera: level view at 0.60 m so it frames the plant rows, not the floor
The camera was tipped 0.15 rad down at 0.55 m, but ripe fruit sits at
~0.85-0.95 m on the gutters -- above the camera -- so the downward view
showed mostly dark ground and missed the berries. Level it and raise it to
0.60 m; the plant rows now fill the frame.

Co-Authored-By: Claude Opus 4.8 <noreply@anthropic.com>
Claude-Session: https://claude.ai/code/session_01Uhu7fuqyazcPGV5GTXJMX5

File: src/youbot_gazebo/urdf/youbot_gz.urdf (robot description, URDF)
Before this commit: robot youbot, 10 links, 9 joints
Joints:
- joint j_camera: origin xyz=0.24 0 0.55 rpy=0 0.15 0 -> xyz=0.24 0 0.60 rpy=0 0 0

Commit message: Phase 4: 5-DOF arm + gripper with scripted pick-and-place
Adds a real articulated arm to the YouBot and an autonomous pick cycle.

- youbot_gz.urdf: replace the dummy arm with a 5-DOF arm (real YouBot
  segment lengths 75/155/135/135/130 mm, reach ~0.9 m to the fruit) plus a
  2-finger parallel gripper (prismatic). One gz JointPositionController per
  joint on <joint>_cmd; gravity off on the arm so poses hold cleanly.
- gz_bridge.yaml: 7 ROS Float64 -> gz Double joint-command bridges.
- arm_node: smooth keyframe pick sequence (stow -> reach -> grasp -> lift ->
  place -> release -> stow, ~7.5 s) on /do_pick; publishes joint commands,
  /joint_states (so robot_state_publisher animates the arm in RViz) and
  /pick_done.
- mission_node: at a patrol waypoint, if ripe_count >= 1 it stops, triggers a
  pick, waits for /pick_done (20 s timeout), then resumes the patrol.
- gazebo.launch.py runs arm_node; setup.py entry point added.

Dimensions match the CAD spec, so a finished FreeCAD model swaps in as
meshes without changing kinematics or control.

Co-Authored-By: Claude Opus 4.8 <noreply@anthropic.com>
Claude-Session: https://claude.ai/code/session_01Uhu7fuqyazcPGV5GTXJMX5

File: src/youbot_gazebo/urdf/youbot_gz.urdf (robot description, URDF)
Before this commit: robot youbot, 10 links, 9 joints
Links:
- removed link arm_base
- removed link arm_seg
- added link arm_link_1, mass 1.0; visual cylinder length=0.075 radius=0.045
- added link arm_link_2, mass 0.8; visual cylinder length=0.155 radius=0.035
- added link arm_link_3, mass 0.6; visual cylinder length=0.135 radius=0.030
- added link arm_link_4, mass 0.4; visual cylinder length=0.135 radius=0.028
- added link arm_link_5, mass 0.3; visual cylinder length=0.130 radius=0.025
- added link finger_left, mass 0.05; visual box size=0.02 0.012 0.05
- added link finger_right, mass 0.05; visual box size=0.02 0.012 0.05
- added link gripper_base, mass 0.15; visual box size=0.05 0.08 0.03
Joints:
- removed joint j_arm
- removed joint j_arm2
- added joint arm_joint_1: type revolute, parent base_link, child arm_link_1, origin xyz=0.12 0 0.16, axis 0 0 1, limit lower=-2.95 upper=2.95 effort=30 velocity=1.5
- added joint arm_joint_2: type revolute, parent arm_link_1, child arm_link_2, origin xyz=0 0 0.075, axis 0 1 0, limit lower=-1.13 upper=1.57 effort=30 velocity=1.5
- added joint arm_joint_3: type revolute, parent arm_link_2, child arm_link_3, origin xyz=0 0 0.155, axis 0 1 0, limit lower=-2.64 upper=2.55 effort=20 velocity=1.5
- added joint arm_joint_4: type revolute, parent arm_link_3, child arm_link_4, origin xyz=0 0 0.135, axis 0 1 0, limit lower=-1.79 upper=1.79 effort=15 velocity=1.5
- added joint arm_joint_5: type revolute, parent arm_link_4, child arm_link_5, origin xyz=0 0 0.135, axis 0 0 1, limit lower=-2.92 upper=2.92 effort=10 velocity=1.5
- added joint gripper_left: type prismatic, parent gripper_base, child finger_left, origin xyz=0 0.015 0.015, axis 0 1 0, limit lower=0.0 upper=0.035 effort=20 velocity=0.2
- added joint gripper_mount: type fixed, parent arm_link_5, child gripper_base, origin xyz=0 0 0.130
- added joint gripper_right: type prismatic, parent gripper_base, child finger_right, origin xyz=0 -0.015 0.015, axis 0 -1 0, limit lower=0.0 upper=0.035 effort=20 velocity=0.2

Commit message: Arm: mount on a raised column facing the plant row (reach the fruit)
The arm pointed down the empty aisle and was too low to reach the ~0.9 m
fruit (shoulder at 0.16 m, reach ~0.6 m).

- Add a 0.39 m pedestal column: the shoulder now sits at ~0.55 m, so the
  arm comfortably reaches fruit height.
- Rotate the arm base 90 deg so it faces the +Y plant row beside the robot
  instead of forward down the aisle.
- Retune the pick keyframes to swing out into the row, grasp at fruit
  height, then swing back over the robot to drop.

Co-Authored-By: Claude Opus 4.8 <noreply@anthropic.com>
Claude-Session: https://claude.ai/code/session_01Uhu7fuqyazcPGV5GTXJMX5

File: src/youbot_gazebo/urdf/youbot_gz.urdf (robot description, URDF)
Before this commit: robot youbot, 16 links, 15 joints
Links:
- added link pedestal, mass 1.5; visual cylinder length=0.39 radius=0.05
Joints:
- added joint j_pedestal: type fixed, parent base_link, child pedestal, origin xyz=0.12 0 0.16
- joint arm_joint_1: origin xyz=0.12 0 0.16 -> xyz=0.12 0 0.55 rpy=0 0 1.5708

Commit message: Option A: real harvest - held strawberry, collection basket, count
Makes the pick more than a gesture.

- youbot_gz.urdf: add a collection basket (open crate) on the rear plate,
  visible in Gazebo and RViz.
- arm_node: a red strawberry marker rides the gripper frame from grasp to
  release, then the released fruit joins a growing pile in the basket
  (RViz markers on /harvest_markers); publishes /harvest_count and logs the
  running total.

Note: the held fruit + pile are RViz markers (Gazebo does not render ROS
markers); the basket itself shows in Gazebo. A gz DetachableJoint would make
the fruit physically stick to the gripper in the Gazebo 3D view.

Co-Authored-By: Claude Opus 4.8 <noreply@anthropic.com>
Claude-Session: https://claude.ai/code/session_01Uhu7fuqyazcPGV5GTXJMX5

File: src/youbot_gazebo/urdf/youbot_gz.urdf (robot description, URDF)
Before this commit: robot youbot, 17 links, 16 joints
Links:
- added link basket, mass 0.2; visual box size=0.01 0.28 0.12; visual box size=0.01 0.28 0.12
Joints:
- added joint j_basket: type fixed, parent base_link, child basket, origin xyz=-0.13 0 0.19

Commit message: Camera faces the +Y row (same side as the arm): no more picking in the void
The camera looked forward down the aisle while the arm reached sideways
(+Y), so the robot stopped on fruit seen far ahead and the arm deployed into
empty space -- picking in the void, especially at aisle ends.

Turn the camera to look LEFT (+Y), the same row the arm harvests. Now the
robot only stops when a fruit is actually beside it, the arm reaches toward
that fruit, and the camera watches the arm approach it. At aisle ends the
+Y side is a wall, so it no longer picks where there is nothing.

Co-Authored-By: Claude Opus 4.8 <noreply@anthropic.com>
Claude-Session: https://claude.ai/code/session_01Uhu7fuqyazcPGV5GTXJMX5

File: src/youbot_gazebo/urdf/youbot_gz.urdf (robot description, URDF)
Before this commit: robot youbot, 18 links, 17 joints
Joints:
- joint j_camera: origin xyz=0.24 0 0.60 rpy=0 0 0 -> xyz=0.18 0.14 0.60 rpy=0 0 1.5708

Commit message: Tilt the camera up 0.5 rad to see the fruit on top of the gutter
Facing +Y level, the camera only saw the brown 0.8 m gutter wall (the fruit
sits on top, above the sight line). Pitch it up ~0.5 rad so it looks over the
gutter edge at the strawberries the arm reaches for.

Co-Authored-By: Claude Opus 4.8 <noreply@anthropic.com>
Claude-Session: https://claude.ai/code/session_01Uhu7fuqyazcPGV5GTXJMX5

File: src/youbot_gazebo/urdf/youbot_gz.urdf (robot description, URDF)
Before this commit: robot youbot, 18 links, 17 joints
Joints:
- joint j_camera: origin xyz=0.18 0.14 0.60 rpy=0 0 1.5708 -> xyz=0.18 0.14 0.60 rpy=0 -0.5 1.5708

Commit message: Raise camera to 0.78 m + better angle; smoother alignment, fewer skips
Camera: 0.60 -> 0.78 m with a gentler up-tilt (0.28 rad) so the berries fill
the frame instead of the brown gutter wall; mast extended to match.

Alignment: proportional centring (slows as it approaches, ALIGN_KP with
vmin/vmax) instead of constant creep, and the drive-sense auto-flip now checks
over a 1.2 s window (robust to noise) rather than per-tick. Relax CENTER_TOL to
0.15 and cut PICK_SPACING to 0.7 m so it picks almost every plant instead of
skipping fruit.

Co-Authored-By: Claude Opus 4.8 <noreply@anthropic.com>
Claude-Session: https://claude.ai/code/session_01Uhu7fuqyazcPGV5GTXJMX5

File: src/youbot_gazebo/urdf/youbot_gz.urdf (robot description, URDF)
Before this commit: robot youbot, 18 links, 17 joints
Links:
- link mast: geometry visual cylinder length=0.62 radius=0.015
Joints:
- joint j_camera: origin xyz=0.18 0.14 0.60 rpy=0 -0.5 1.5708 -> xyz=0.18 0.14 0.78 rpy=0 -0.28 1.5708

Commit message: Assemble the real CAD robot: body + 4 mecanum wheel meshes in Gazebo
Replace the primitive body box and wheel cylinders with your FreeCAD meshes:
- meshes/base.stl, wheel_A.stl, wheel_B.stl (mm; scaled 0.001 in URDF).
- Body: yaw -90 deg so its 580 mm length faces +X; wheels: roll 90 deg so the
  axle is along Y, shifted to centre the 50 mm width, placed at the body's
  four arches (+/-0.225, +/-0.19, r 0.054). Handedness A on FL/RR, B on FR/RL.
- Visual-only swap (no collision) -> navigation and picking are unchanged.
- launch: set GZ_SIM_RESOURCE_PATH so gz resolves the package:// mesh URIs;
  setup.py installs the meshes.

Co-Authored-By: Claude Opus 4.8 <noreply@anthropic.com>
Claude-Session: https://claude.ai/code/session_01Uhu7fuqyazcPGV5GTXJMX5

File: src/youbot_gazebo/urdf/youbot_gz.urdf (robot description, URDF)
Before this commit: robot youbot, 18 links, 17 joints
Links:
- link base_link: geometry visual mesh filename=package://youbot_gazebo/meshes/base.stl scale=0.001 0.001 0.001
- link wheel_fl: geometry visual mesh filename=package://youbot_gazebo/meshes/wheel_A.stl scale=0.001 0.001 0.001
- link wheel_fr: geometry visual mesh filename=package://youbot_gazebo/meshes/wheel_B.stl scale=0.001 0.001 0.001
- link wheel_rl: geometry visual mesh filename=package://youbot_gazebo/meshes/wheel_B.stl scale=0.001 0.001 0.001
- link wheel_rr: geometry visual mesh filename=package://youbot_gazebo/meshes/wheel_A.stl scale=0.001 0.001 0.001
Joints:
- joint j_fl: origin xyz=0.228 0.178 0.05 -> xyz=0.225 0.19 0.054
- joint j_fr: origin xyz=0.228 -0.178 0.05 -> xyz=0.225 -0.19 0.054
- joint j_rl: origin xyz=-0.228 0.178 0.05 -> xyz=-0.225 0.19 0.054
- joint j_rr: origin xyz=-0.228 -0.178 0.05 -> xyz=-0.225 -0.19 0.054

Commit message: SLAM corridor fix: basket out of the lidar plane + low-gain correction fusion
Field log analysis: SLAM was excellent while driving near the spawn (0.08 m,
better than odometry) then locked in the long aisle at ~30% of driving speed
and plateaued at 6.5 m offset. Root cause: the basket walls (z 0.19-0.31)
filled the lidar plane (z 0.20) across ~150 deg of the rear, and the
self-hit filter rightly dropped those beams, leaving the robot blind
BACKWARDS -- exactly the direction that pins along-corridor position against
the already-mapped wall behind.

* URDF: basket raised on four legs (walls now z 0.26-0.38, above the plane;
  thin legs stay under the 0.35 m self-hit filter). Same lesson as a real
  robot: mount the lidar clear of the chassis or the chassis becomes the map.
* slam_node: corrections applied at 35% gain (complementary-filter style):
  odometry drift is a few mm per matched step so tracking is unaffected,
  while any residual matcher bias is divided by ~3 instead of integrating.

Bench (stationary pick periods included): mean 0.050 m / max 0.084 m.

Co-Authored-By: Claude Opus 4.8 <noreply@anthropic.com>
Claude-Session: https://claude.ai/code/session_01Uhu7fuqyazcPGV5GTXJMX5

File: src/youbot_gazebo/urdf/youbot_gz.urdf (robot description, URDF)
Before this commit: robot youbot, 18 links, 17 joints
Links:
- link basket: geometry visual box size=0.01 0.28 0.12; visual box size=0.01 0.28 0.12
Joints:
- joint j_basket: origin xyz=-0.13 0 0.19 -> xyz=-0.13 0 0.26

Commit message: Unblock the robot: one fence, a swept-corridor brake, and a lidar that can see forward
The last run harvested 29 berries with SLAM at 0.04 m, then spent most of a lap
pinned around (-4.3, +1.5) with "Stuck -- backing off and turning" and a goal
timeout on (-3.80, +0.60). Three faults, all in the containment layer:

1. Two fences with different boundaries. navigation_node pushed back inside
   from 0.25 m BEFORE the bound while safety_node only reacted past it, and
   flank recentring pushed the other way below y = 1.68. That left a 0.17 m
   band where two bang-bang controls fought each other -- exactly the observed
   x = -4.30, y = 1.31..1.67 ping-pong. The fence and the brake now live only
   in safety_node; navigation_node keeps the stuck detector, which is the one
   thing only the path follower can judge.

2. A cone brake that measured the wrong thing. A +/-0.55 rad cone reaches
   0.28 m sideways at half a metre, so a beam grazing a gutter the robot was
   legitimately driving PAST came back short and braked it in open corridor;
   and the raw range along an oblique beam overstates how soon we arrive.
   Replaced by the swept rectangle: projected on the direction of travel, how
   far ahead is the nearest return inside the robot's own width. Flank
   clearance is measured the same way, over a band level with the base rather
   than a cone that picks up whatever is diagonally ahead. Recentring is now
   proportional, only acts while translating, and only pushes toward a side
   that has room -- in a passage narrower than 2*side_min it holds still
   instead of shoving into the opposite wall.

3. The robot was blind forward. gpu_lidar ray-casts the visuals, and the arm
   column (r = 0.05 at x = 0.12) crossed the sensor plane: it walled off
   +/-25 deg of the forward view. Those returns land at 0.07 m and are dropped
   as self-hits, so the forward brake was left reading only the oblique beams
   past 25 deg -- the ones that graze the gutters. A thin collar through the
   lidar plane, the way a real mast is cut away around a scanner, drops the
   blind sector to +/-6 deg.

Also moved the spawn to (-4.40, 1.85): -4.6 sat outside the fence, so the
guard opened every run by shoving the robot back in.

Checked offline by ray-casting a 2D model of the greenhouse at the poses from
the log: at (-4.35, 1.60) heading east the recentring now pushes +0.04 m/s
north and dies out by y = 1.70, with the fence silent until 2.15 -- a 0.45 m
stable band instead of the old 0.17 m trap. Centred in an aisle both flanks
read 0.40 m and nothing is applied; 0.15 m off-centre it corrects at 0.02 m/s.

Co-Authored-By: Claude Opus 5 <noreply@anthropic.com>
Claude-Session: https://claude.ai/code/session_01Uhu7fuqyazcPGV5GTXJMX5

File: src/youbot_gazebo/urdf/youbot_gz.urdf (robot description, URDF)
Before this commit: robot youbot, 18 links, 17 joints
Links:
- link pedestal: geometry visual cylinder length=0.10 radius=0.012; visual cylinder length=0.29 radius=0.05
