Commit message: Fix robot visibility + SLAM drift: inline colors, correction clamping
Visibility: every URDF <material> reference now carries an inline <color>
so sdformat's URDF→SDF converter always has explicit RGBA values, even if
global material name resolution fails (which made the robot invisible).
A primitive orange box is added to base_link as a guaranteed fallback
when mesh loading fails.

SLAM: three layers of correction limiting to stop the scan matcher from
pulling the pose away from truth:
  1. min_gain raised 0.01 → 0.05 (require real score improvement, not noise)
  2. Per-scan correction clamped to ±0.04 m (lin) and ±0.03 rad (ang)
  3. Trust gate in slam_node rejects corrections > max(0.03 m, 3× odom step)
     and skips map update on rejection (prevents smearing)

Logging improved: shows instantaneous error, accepted/rejected correction
counts per reporting period.

File: src/youbot_gazebo/urdf/youbot_gz.urdf (robot description, URDF)
Before this commit: robot youbot, 19 links, 18 joints
Links:
- link base_link: geometry visual box size=0.58 0.37 0.12; visual mesh filename=package://youbot_gazebo/meshes/base.stl scale=0.001 0.001 0.001
