Commit message: cloud_agri: park the robot AT the plant, and aim the camera at it
Two defects, one visible in every photograph and neither obviously wrong.

THE CAMERA WAS AIMED FROM THE WRONG POINT. pan_for() computed the
bearing from the STATION -- the boom tip, under the floor camera --
while the lens sits on the mast, CAMERA_LEVER_X = 0.32 m behind it.
The two points see the plant 30.2 degrees apart. Against a 69-degree
field of view that is 0.9 of a half-frame, so the plant stayed just
inside the picture at every station and 48 photographs a run went on
looking acceptable. pan_for now projects from the lens, and the check
that used to assert "+/-90 degrees" -- a statement about the cross,
not about the camera -- now asserts the ray actually hits the plant.

THE CHASSIS WAS HALF A METRE DOWN THE AISLE FROM THE PLANT. The cross
sat at the plant's own x, and the cross is under the boom tip, so
base_link ended up 0.50 m along the row from the plant it was
measuring. Every reading was still filed correctly, which is why
nothing caught it. Crosses now sit at plant_x + SENSOR_OFFSET_X, which
puts base_link exactly on the plant: the robot straddles it, the floor
camera still lies over the cross, and the residual aiming error is
0.00 degrees at all 48 stations.

That geometry needs 108.1 degrees of pan and Phase B built the head
with 90. make_robot.py widens the limit to 125 during generation --
Phase C generates its own robot and must not write into Phase B -- and
reads the mast's mounting x back out of the source to assert it
matches the constant the aiming maths uses.

Also, from the same review:

  * A measurement table at /table: one row per PLANT, right-hand
    station and its media links first, then the left-hand station, on
    the same line. store/plants.csv is written in that same shape, so
    the file and the page are read the same way. It is a second file
    rather than a reshaped measurements.csv, because that one is the
    audit trail: three visits to a station are three rows there, and
    collapsing them would discard the history.

  * The photograph and the QR code now render at the same size. The
    photo is letterboxed rather than cropped -- cropping it to tidy a
    layout throws away the evidence it exists to carry.

An unmeasured side exports as an empty cell, never a zero.

413 checks pass.

Co-Authored-By: Claude Opus 5 <noreply@anthropic.com>
Claude-Session: https://claude.ai/code/session_01Uhu7fuqyazcPGV5GTXJMX5

File: cloud_agri/urdf/youbot_agri.urdf (robot description, URDF)
Before this commit: robot youbot, 21 links, 20 joints
Joints:
- joint j_camera_pan: limit lower=-1.5708 upper=1.5708 effort=4.0 velocity=1.5 -> lower=-2.1817 upper=2.1817 effort=4.0 velocity=1.5
